File: PCB/TumTa.brd (EAGLE design)
At the start: 16 parts

Commit message: v0_2_4
Parts:
- added C3, C4, C5, C6: (no value), SparkFun-Passives:CPOL-RADIAL-10UF-25V
- moved TA 62.0 mm to (76.0, 58.0), turned to 0 degrees
- moved CAL_TA 56.1 mm to (77.1, 49.9)
- moved C2 38.6 mm to (80.0, 28.0), turned to 0 degrees
- moved LED1(VERDE) 37.1 mm to (43.0, 26.0)
- moved LED2(AMARELO) 37.1 mm to (43.0, 39.0)
- moved SWITCH_STANDBY 37.0 mm to (43.0, 13.0)
- moved C1 36.1 mm to (80.0, 32.0), turned to 0 degrees
- moved CAL_TETO 33.5 mm to (66.5, 54.9)
- moved R1 33.2 mm to (46.0, 27.0)
- moved R4 33.2 mm to (46.0, 18.0), turned to 90 degrees
- moved JP1 33.2 mm to (74.9, 25.4)
- moved R2 33.0 mm to (46.0, 39.0)
- moved FIO_SHIELD 33.0 mm to (61.0, 27.9)
- moved FL1 23.0 mm to (10.2, 12.7)
- moved TUM 14.0 mm to (52.0, 58.0), turned to 0 degrees
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Connections:
- net N$4 renamed D9
- net N$5 renamed D10
- removed net 3.3V: CAL_TA.1, CAL_TUM.1
- removed net N$1: FIO_SHIELD.9, R4.2
- removed net N$11: FIO_SHIELD.24
- removed net N$12: C2.1, CAL_TA.2, TA.1
- removed net N$9: C1.1, CAL_TUM.2, FIO_SHIELD.22, TUM.1
- new net A0: C1.1, C2.1, C3.1, CAL_TUM.2, FIO_SHIELD.21, TUM.1
- new net A1: C4.1, C5.1, C6.1, CAL_TA.2, FIO_SHIELD.22, TA.1
- new net D6: FIO_SHIELD.7, R4.2
- net 3V3: now also CAL_TA.1, CAL_TUM.1
- net GND: now also C3.2, C4.2, C5.2, C6.2
Routing:
- net GND: track 174.6 -> 0.00 mm
- net 3V3: track 90.3 -> 0.00 mm
- net AREF: track 65.6 -> 0.00 mm
- net N$9: track 53.5 -> 0.00 mm
- net N$12: track 48.1 -> 0.00 mm
- net 3.3V: track 25.2 -> 0.00 mm
- net N$1: track 14.6 -> 0.00 mm
- net N$2: track 11.7 -> 0.00 mm
- net N$7: track 7.88 -> 0.00 mm
- net N$3: track 7.47 -> 0.00 mm
- net D9: track 5.30 -> 0.00 mm
- net D10: track 3.43 -> 0.00 mm
- net RXI: track 2.96 -> 0.00 mm
- net DTR: track 2.96 -> 0.00 mm
- net TXO: track 2.96 -> 0.00 mm
Other:
- board outline added: 100 x 80 mm

Commit message: v0_2_10
Parts:
- removed C1, C3, C4, C6: (no value), SparkFun-Passives:CPOL-RADIAL-10UF-25V
- removed CAL_TA, CAL_TETO, CAL_TUM: TRIMPOT_MULTIVOLTAS, SparkFun-Electromechanical:TRIMPOT_MULTIVOLTAS
- removed FL1: FRAME-LETTER_BATEBIT, SparkFun-Retired:BATEBIT
- removed LED1(VERDE): SCREWTERMINAL-25MM, SparkFun-Connectors:SCREWTERMINAL-5MM-2
- removed R1: 100, SparkFun-Resistors:0603-RES
- added AREF, R3: (no value), SparkFun-Electromechanical:TRIM_POT_BR
- added R5: 4.7K, SparkFun-Resistors:0603-RES
- added S1: (no value), SparkFun-Electromechanical:SWITCH-SPDT
- added TA_CALIB, TUM_CALIB: TRIMPOT_MULTIVOLTAS, SparkFun-Electromechanical:TRIMPOT_MULTIVOLTAS
- moved C2 38.5 mm to (44.0, 41.5), flipped to the top, turned to 180 degrees
- moved LED2(AMARELO) 37.9 mm to (78.8, 26.6), flipped to the top
- moved SWITCH_STANDBY 35.7 mm to (78.7, 14.6), flipped to the top
- moved JP1 33.4 mm to (43.5, 36.5), flipped to the top
- moved R2 32.3 mm to (76.1, 27.2), turned to 90 degrees
- moved R4 30.4 mm to (76.2, 14.4), turned to 270 degrees
- moved TUM 6.29 mm to (46.9, 54.3), flipped to the top, turned to 180 degrees
- moved TA 6.14 mm to (80.9, 54.3), flipped to the top, turned to 180 degrees
- moved C5 2.93 mm to (79.4, 40.1), flipped to the top, turned to 180 degrees
- flipped FIO_SHIELD to the top
Connections:
- removed net D6: FIO_SHIELD.7, R4.2
- removed net D9: FIO_SHIELD.10, R1.2
- new net N$1: FIO_SHIELD.28, R3.2
- new net N$4: R5.2, S1.3
- net 3V3: now also AREF.3, R3.3, R4.2, R5.1, TA.2, TA_CALIB.3, TUM.2, TUM_CALIB.3; no longer CAL_TA.1, CAL_TETO.3, CAL_TUM.1
- net A0: now also TUM_CALIB.2; no longer C1.1, C3.1, CAL_TUM.2
- net A1: now also TA_CALIB.2; no longer C4.1, C6.1, CAL_TA.2
- net AREF: now also AREF.2; no longer CAL_TETO.2
- net D10: now also FIO_SHIELD.7; no longer FIO_SHIELD.11
- net GND: now also AREF.1, R3.1, S1.1, TA_CALIB.1, TUM_CALIB.1; no longer C1.2, C3.2, C4.2, C6.2, CAL_TETO.1, LED1(VERDE).2, TA.2, TUM.2
- net N$2: now also FIO_SHIELD.3
- net N$3: now also FIO_SHIELD.13, S1.2; no longer LED1(VERDE).1, R1.1
Routing:
- net GND: track 0.00 -> 203.5 mm
- net 3V3: track 0.00 -> 180.1 mm
- net A1: track 0.00 -> 90.2 mm
- net N$3: track 0.00 -> 67.4 mm
- net A0: track 0.00 -> 40.3 mm
- net N$1: track 0.00 -> 17.8 mm
- net AREF: track 0.00 -> 16.3 mm
- net TXO: track 0.00 -> 14.6 mm
- net DTR: track 0.00 -> 14.2 mm
- net RXI: track 0.00 -> 13.9 mm
- net N$2: track 0.00 -> 7.80 mm
- net N$4: track 0.00 -> 4.48 mm
- net D10: track 0.00 -> 3.43 mm
- net N$7: track 0.00 -> 2.83 mm
- added copper zone on layer 16, net GND
Other:
- board size 100 x 80 mm -> 49.8 x 50.9 mm

Commit message: v0_2_3
Parts:
- removed AREF, R3: (no value), SparkFun-Electromechanical:TRIM_POT_BR
- removed C5: (no value), SparkFun-Passives:CPOL-RADIAL-10UF-25V
- removed R5: 4.7K, SparkFun-Resistors:0603-RES
- removed S1: (no value), SparkFun-Electromechanical:SWITCH-SPDT
- removed TA_CALIB, TUM_CALIB: TRIMPOT_MULTIVOLTAS, SparkFun-Electromechanical:TRIMPOT_MULTIVOLTAS
- added C1: (no value), SparkFun-Passives:CPOL-RADIAL-10UF-25V
- added CAL_TA, CAL_TETO, CAL_TUM: TRIMPOT_MULTIVOLTAS, SparkFun-Electromechanical:TRIMPOT_MULTIVOLTAS
- added FL1: FRAME-LETTER_BATEBIT, SparkFun-Retired:BATEBIT
- added LED1(VERDE): SCREWTERMINAL-25MM, SparkFun-Connectors:SCREWTERMINAL-5MM-2
- added R1: 100, SparkFun-Resistors:0603-RES
- moved LED2(AMARELO) 74.4 mm to (6.00, 42.0), flipped to the bottom
- moved SWITCH_STANDBY 72.7 mm to (6.00, 14.0), flipped to the bottom
- moved TA 67.0 mm to (14.0, 58.0), flipped to the bottom
- moved R2 64.2 mm to (13.0, 39.0), turned to 270 degrees
- moved R4 63.7 mm to (13.0, 22.0), turned to 90 degrees
- moved FIO_SHIELD 33.0 mm to (28.0, 28.0), flipped to the bottom
- moved JP1 11.0 mm to (41.7, 25.6), flipped to the bottom
- moved TUM 9.65 mm to (38.0, 58.0), flipped to the bottom
- moved C2 0.49 mm to (44.0, 42.0), flipped to the bottom, turned to 270 degrees
Connections:
- removed net A0: C2.1, FIO_SHIELD.21, TUM.1, TUM_CALIB.2
- removed net A1: C5.1, FIO_SHIELD.22, TA.1, TA_CALIB.2
- removed net D10: FIO_SHIELD.7, R2.2
- removed net N$1: FIO_SHIELD.28, R3.2
- new net 3.3V: CAL_TA.1, CAL_TUM.1
- new net N$11: FIO_SHIELD.24
- new net N$12: C2.1, CAL_TA.2, TA.1
- new net N$5: FIO_SHIELD.11, R2.2
- new net N$9: C1.1, CAL_TUM.2, FIO_SHIELD.22, TUM.1
- net 3V3: now also CAL_TETO.3; no longer AREF.3, R3.3, R4.2, R5.1, TA.2, TA_CALIB.3, TUM.2, TUM_CALIB.3
- net AREF: now also CAL_TETO.2; no longer AREF.2
- net GND: now also C1.2, CAL_TETO.1, LED1(VERDE).2, TA.2, TUM.2; no longer AREF.1, C5.2, R3.1, S1.1, TA_CALIB.1, TUM_CALIB.1
- net N$2: no longer FIO_SHIELD.3
- net N$3: now also LED1(VERDE).1, R1.1; no longer FIO_SHIELD.13, S1.2
- net N$4: now also FIO_SHIELD.10, R1.2; no longer R5.2, S1.3
Routing:
- net A1: track 90.2 -> 0.00 mm
- net 3V3: track 180.1 -> 93.6 mm
- net N$3: track 67.4 -> 7.47 mm
- net N$9: track 0.00 -> 56.1 mm
- net AREF: track 16.3 -> 66.0 mm
- net N$12: track 0.00 -> 46.8 mm
- net A0: track 40.3 -> 0.00 mm
- net 3.3V: track 0.00 -> 22.1 mm
- net GND: track 203.5 -> 182.9 mm
- net N$1: track 17.8 -> 0.00 mm
- net TXO: track 14.6 -> 2.96 mm
- net DTR: track 14.2 -> 2.96 mm
- net RXI: track 13.9 -> 2.96 mm
- net N$7: track 2.83 -> 7.88 mm
- net D10: track 3.43 -> 0.00 mm
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Other:
- board outline removed

Commit message: v0_2_4
Parts:
- added C3, C4, C5, C6: (no value), SparkFun-Passives:CPOL-RADIAL-10UF-25V
- moved TA 62.0 mm to (76.0, 58.0), turned to 0 degrees
- moved CAL_TA 56.1 mm to (77.1, 49.9)
- moved C2 38.6 mm to (80.0, 28.0), turned to 0 degrees
- moved LED1(VERDE) 37.1 mm to (43.0, 26.0)
- moved LED2(AMARELO) 37.1 mm to (43.0, 39.0)
- moved SWITCH_STANDBY 37.0 mm to (43.0, 13.0)
- moved C1 36.1 mm to (80.0, 32.0), turned to 0 degrees
- moved CAL_TETO 33.5 mm to (66.5, 54.9)
- moved R1 33.2 mm to (46.0, 27.0)
- moved R4 33.2 mm to (46.0, 18.0)
- moved JP1 33.2 mm to (74.9, 25.4)
- moved R2 33.0 mm to (46.0, 39.0)
- moved FIO_SHIELD 33.0 mm to (61.0, 27.9)
- moved FL1 23.0 mm to (10.2, 12.7)
- moved TUM 14.0 mm to (52.0, 58.0), turned to 0 degrees
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Connections:
- net N$4 renamed D9
- net N$5 renamed D10
- removed net 3.3V: CAL_TA.1, CAL_TUM.1
- removed net N$11: FIO_SHIELD.24
- removed net N$12: C2.1, CAL_TA.2, TA.1
- removed net N$9: C1.1, CAL_TUM.2, FIO_SHIELD.22, TUM.1
- new net A0: C1.1, C2.1, C3.1, CAL_TUM.2, FIO_SHIELD.21, TUM.1
- new net A1: C4.1, C5.1, C6.1, CAL_TA.2, FIO_SHIELD.22, TA.1
- new net D6: FIO_SHIELD.7, R4.2
- net 3V3: now also CAL_TA.1, CAL_TUM.1
- net GND: now also C3.2, C4.2, C5.2, C6.2
Routing:
- net GND: track 182.9 -> 0.00 mm
- net 3V3: track 93.6 -> 0.00 mm
- net AREF: track 66.0 -> 0.00 mm
- net N$9: track 56.1 -> 0.00 mm
- net N$12: track 46.8 -> 0.00 mm
- net 3.3V: track 22.1 -> 0.00 mm
- net N$2: track 10.0 -> 0.00 mm
- net N$7: track 7.88 -> 0.00 mm
- net N$3: track 7.47 -> 0.00 mm
- net D9: track 5.30 -> 0.00 mm
- net D10: track 3.43 -> 0.00 mm
- net RXI: track 2.96 -> 0.00 mm
- net DTR: track 2.96 -> 0.00 mm
- net TXO: track 2.96 -> 0.00 mm
- removed copper zone on layer 16, net GND
Other:
- board outline added: 100 x 80 mm

Commit message: v0_2_5
Parts:
- moved CAL_TETO 44.6 mm to (78.2, 11.9), turned to 90 degrees
- moved TA 5.00 mm to (71.0, 58.0), turned to 180 degrees
- moved TUM 5.00 mm to (47.0, 58.0), turned to 180 degrees
- moved C4 1.00 mm to (80.0, 46.0)
- moved C5 1.00 mm to (80.0, 42.0)
- moved C6 1.00 mm to (80.0, 38.0)
- moved CAL_TA 1.00 mm to (77.1, 48.9)
- moved CAL_TUM 1.00 mm to (55.2, 49.0)
- moved R2 1.00 mm to (46.0, 38.0)
- moved R4 1.00 mm to (46.0, 17.0)
- moved JP1 0.14 mm to (74.8, 25.5)
Routing:
- net GND: track 0.00 -> 154.4 mm
- net 3V3: track 0.00 -> 138.6 mm
- net A0: track 0.00 -> 55.5 mm
- net A1: track 0.00 -> 34.8 mm
- net D6: track 0.00 -> 11.6 mm
- net D9: track 0.00 -> 9.30 mm
- net AREF: track 0.00 -> 9.22 mm
- net N$2: track 0.00 -> 4.40 mm
- net D10: track 0.00 -> 3.70 mm
- net RXI: track 0.00 -> 3.23 mm
- net TXO: track 0.00 -> 3.20 mm
- net DTR: track 0.00 -> 3.17 mm
- net N$3: track 0.00 -> 3.06 mm
- net N$7: track 0.00 -> 3.04 mm

Commit message: v0_2_6
Parts:
- moved C1 16.8 mm to (64.0, 27.0)
- moved C2 16.8 mm to (64.0, 23.0)
- moved C3 16.8 mm to (64.0, 19.0)
- moved C4 16.8 mm to (64.0, 41.0)
- moved C5 16.8 mm to (64.0, 37.0)
- moved C6 16.8 mm to (64.0, 33.0)
- moved CAL_TETO 16.8 mm to (62.2, 6.90)
- moved CAL_TUM 16.8 mm to (39.2, 44.0)
- moved FIO_SHIELD 16.8 mm to (45.0, 22.9)
- moved JP1 16.8 mm to (58.8, 20.5)
- moved LED1(VERDE) 16.8 mm to (27.0, 21.0)
- moved LED2(AMARELO) 16.8 mm to (27.0, 34.0)
- moved R1 16.8 mm to (30.0, 22.0)
- moved R2 16.8 mm to (30.0, 33.0)
- moved R4 16.8 mm to (30.0, 12.0)
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Routing:
- net 3V3: track 138.6 -> 110.8 mm
- net A0: track 55.5 -> 65.9 mm
- net GND: track 154.4 -> 160.8 mm
- net D6: track 11.6 -> 12.6 mm
- added copper zone on layer 16, net GND
Other:
- board text added: "23/06/2015"
- board text added: "Joao Tragtenberg"
- board text added: "Recife"
- board text added: "TumTa"
- board text added: "v0.2.6"

Commit message: v0_2_7
Parts:
- removed CAL_TETO: TRIMPOT_MULTIVOLTAS, SparkFun-Electromechanical:TRIMPOT_MULTIVOLTAS
- added R3: (no value), SparkFun-Electromechanical:TRIM_POT_PTH
- moved R2 16.8 mm to (46.0, 38.2)
- moved C1 16.8 mm to (80.0, 32.0)
- moved C2 16.8 mm to (80.0, 28.0)
- moved C3 16.8 mm to (80.0, 24.0)
- moved C4 16.8 mm to (80.0, 46.0)
- moved C5 16.8 mm to (80.0, 42.0)
- moved C6 16.8 mm to (80.0, 38.0)
- moved CAL_TUM 16.8 mm to (55.2, 49.0)
- moved FIO_SHIELD 16.8 mm to (61.0, 27.9)
- moved JP1 16.8 mm to (74.8, 25.5)
- moved LED1(VERDE) 16.8 mm to (43.0, 26.0)
- moved LED2(AMARELO) 16.8 mm to (43.0, 39.0)
- moved R4 16.8 mm to (46.0, 17.0)
- moved SWITCH_STANDBY 16.8 mm to (43.0, 13.0)
- moved TA 16.8 mm to (71.0, 58.0)
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Connections:
- net 3V3: now also R3.3, TA.2, TUM.2; no longer CAL_TA.1, CAL_TETO.3, CAL_TUM.1
- net AREF: now also R3.2; no longer CAL_TETO.2
- net GND: now also CAL_TA.1, CAL_TUM.1, R3.1; no longer CAL_TETO.1, TA.2, TUM.2
Routing:
- net GND: track 160.8 -> 188.7 mm
- net AREF: track 9.22 -> 5.65 mm
- net 3V3: track 110.8 -> 107.8 mm
- net D6: track 12.6 -> 11.8 mm
Other:
- board text removed: "23/06/2015"
- board text removed: "Joao Tragtenberg"
- board text removed: "Recife"
- board text removed: "TumTa"
- board text removed: "v0.2.6"

Commit message: v0_2_8
Parts:
- removed CAL_TA, CAL_TUM: TRIMPOT_MULTIVOLTAS, SparkFun-Electromechanical:TRIMPOT_MULTIVOLTAS
- removed R3: (no value), SparkFun-Electromechanical:TRIM_POT_PTH
- added AREF, TA_CALIB, TUM_CALIB: (no value), SparkFun-Electromechanical:TRIM_POT_BR
- moved TA 7.00 mm to (77.0, 54.4)
- moved TUM 5.45 mm to (43.0, 54.3)
- moved R1 2.00 mm to (46.0, 28.8)
Connections:
- new net 3.3V: TA.2, TA_CALIB.3, TUM.2, TUM_CALIB.3
- net 3V3: now also AREF.3; no longer R3.3, TA.2, TUM.2
- net A0: now also TUM_CALIB.2; no longer CAL_TUM.2
- net A1: now also TA_CALIB.2; no longer CAL_TA.2
- net AREF: now also AREF.2; no longer R3.2
- net GND: now also AREF.1, TA_CALIB.1, TUM_CALIB.1; no longer CAL_TA.1, CAL_TUM.1, R3.1
Routing:
- net 3V3: track 107.8 -> 39.0 mm
- net 3.3V: track 0.00 -> 38.9 mm
- net GND: track 188.7 -> 193.7 mm
- net AREF: track 5.65 -> 9.02 mm
- net A0: track 66.1 -> 64.1 mm
- net D9: track 9.41 -> 7.44 mm
- net A1: track 34.7 -> 36.2 mm
- net N$3: track 3.02 -> 3.81 mm
