File: PCB/TumTa.brd (EAGLE design)
At the start: 100 x 80 mm, 20 parts

Commit message: v0_2_9
Parts:
- removed C1, C2, C3, C4, C5, C6: (no value), SparkFun-Passives:CPOL-RADIAL-10UF-25V
- removed FL1: FRAME-LETTER_BATEBIT, SparkFun-Retired:BATEBIT
- removed JP1: (no value), SparkFun-Connectors:1X06
- removed LED1(VERDE): SCREWTERMINAL-25MM, SparkFun-Connectors:SCREWTERMINAL-5MM-2
- removed R1: 100, SparkFun-Resistors:0603-RES
- added C_TA, C_TUM: (no value), SparkFun-Passives:CPOL-RADIAL-10UF-25V
- added FTDI: (no value), SparkFun-Connectors:1X06
- added MODO: (no value), SparkFun-Electromechanical:SWITCH-SPDT
- added R5: 4.7K, SparkFun-Resistors:0603-RES
- added THRESHOLD: (no value), SparkFun-Electromechanical:TRIM_POT_BR
- TA_CALIB, TUM_CALIB: value (none) -> TRIMPOT_MULTIVOLTAS; device SparkFun-Electromechanical:TRIM_POT_BR -> SparkFun-Electromechanical:TRIMPOT_MULTIVOLTAS
- moved TA 36.0 mm to (41.0, 54.4)
- moved TUM 33.0 mm to (76.0, 54.3)
- moved TUM_CALIB 28.2 mm to (84.1, 45.1)
- moved TA_CALIB 22.1 mm to (47.3, 45.2)
- moved LED2(AMARELO) 13.0 mm to (43.0, 26.0)
- moved R2 11.0 mm to (46.0, 27.2), turned to 90 degrees
- moved AREF 4.00 mm to (79.0, 16.0)
- moved R4 3.00 mm to (46.0, 14.0), turned to 270 degrees
- moved SWITCH_STANDBY 1.00 mm to (43.0, 14.0)
Connections:
- removed net 3.3V: TA.2, TA_CALIB.3, TUM.2, TUM_CALIB.3
- removed net D6: FIO_SHIELD.7, R4.2
- removed net D9: FIO_SHIELD.10, R1.2
- new net N$1: FIO_SHIELD.28, THRESHOLD.2
- new net N$4: MODO.3, R5.2
- net 3V3: now also FTDI.4, R4.2, R5.1, TA.2, TA_CALIB.3, THRESHOLD.3, TUM.2, TUM_CALIB.3; no longer JP1.4
- net A0: now also C_TUM.1, FIO_SHIELD.22; no longer C1.1, C2.1, C3.1, FIO_SHIELD.21
- net A1: now also C_TA.1, FIO_SHIELD.21; no longer C4.1, C5.1, C6.1, FIO_SHIELD.22
- net AREF: now also FTDI.5; no longer JP1.5
- net D10: now also FIO_SHIELD.7; no longer FIO_SHIELD.11
- net DTR: now also FTDI.1; no longer JP1.1
- net GND: now also C_TA.2, C_TUM.2, FTDI.6, MODO.1, THRESHOLD.1; no longer C1.2, C2.2, C3.2, C4.2, C5.2, C6.2, JP1.6, LED1(VERDE).2
- net N$2: now also FIO_SHIELD.3
- net N$3: now also FIO_SHIELD.13, MODO.2; no longer LED1(VERDE).1, R1.1
- net RXI: now also FTDI.3; no longer JP1.3
- net TXO: now also FTDI.2; no longer JP1.2
Routing:
- net 3V3: track 39.0 -> 251.5 mm, vias 0 -> 3
- net A1: track 36.2 -> 85.6 mm
- net 3.3V: track 38.9 -> 0.00 mm
- net A0: track 64.1 -> 28.6 mm
- net GND: track 193.7 -> 166.1 mm
- net D6: track 11.6 -> 0.00 mm
- net DTR: track 3.18 -> 12.8 mm
- net TXO: track 3.30 -> 12.8 mm
- net N$3: track 3.81 -> 13.2 mm
- net RXI: track 3.46 -> 12.8 mm
- net AREF: track 9.02 -> 17.8 mm
- net N$1: track 0.00 -> 7.58 mm
- net D9: track 7.44 -> 0.00 mm
- net N$4: track 0.00 -> 3.78 mm, vias 0 -> 1
- net N$2: track 4.61 -> 7.90 mm, vias 0 -> 2
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Other:
- board size 100 x 80 mm -> 49 x 51 mm
- board text added: "BLK"
- board text added: "GRN"

Commit message: v1_0_0
Parts:
- removed AREF, THRESHOLD: (no value), SparkFun-Electromechanical:TRIM_POT_BR
- removed C_TA, C_TUM: (no value), SparkFun-Passives:CPOL-RADIAL-10UF-25V
- removed FTDI: (no value), SparkFun-Connectors:1X06
- removed LED2(AMARELO), SWITCH_STANDBY, TA, TUM: SCREWTERMINAL-25MM, SparkFun-Connectors:SCREWTERMINAL-5MM-2
- removed MODO: (no value), SparkFun-Electromechanical:SWITCH-SPDT
- added C2, C5: (no value), SparkFun-Passives:CPOL-RADIAL-10UF-25V
- added FL1: FRAME-LETTER_BATEBIT, SparkFun-Retired:BATEBIT
- added JP1: (no value), SparkFun-Connectors:1X06
- added JUMPER_CALIB/EXEC, PINS_ON/OFF: (no value), SparkFun-Connectors:1X02
- added LED: (no value), SparkFun-LED:LED5MM
- added ON/OFF: SWITCH, SparkFun-Electromechanical:SWITCH_HH_2POS_3PIN
- added POT_AREF: TRIMPOT_MULTIVOLTAS, SparkFun-Electromechanical:TRIMPOT_MULTIVOLTAS
- added POT_THRESHOLD: (no value), SparkFun-Electromechanical:TRIM_POT_BR
- added STANDBY: SWITCH, SparkFun-Electromechanical:SWITCH_HH_2POS_6PIN
- added U$1: SCREWTERMINAL-5, SparkFun-Connectors:SCREWTERMINAL-0.1"-5_BR
- moved TUM_CALIB 80.6 mm to (16.5, 1.27), flipped to the top, turned to 90 degrees
- moved R5 41.0 mm to (15.2, 36.8), flipped to the top, turned to 0 degrees
- moved TA_CALIB 37.3 mm to (16.5, 24.1), flipped to the top, turned to 90 degrees
- moved R4 30.8 mm to (15.2, 15.2), flipped to the top, turned to 0 degrees
- moved FIO_SHIELD 24.1 mm to (38.1, 20.3), flipped to the top, turned to 270 degrees
- moved R2 14.2 mm to (36.8, 38.1), flipped to the top, turned to 180 degrees
Connections:
- new net 3.3V: POT_THRESHOLD.3
- new net N$6: ON/OFF.P$1, PINS_ON/OFF.2
- new net N$8: ON/OFF.P$2, PINS_ON/OFF.1
- net 3V3: now also JP1.4, POT_AREF.3, U$1.P$2, U$1.P$5; no longer AREF.3, FTDI.4, TA.2, THRESHOLD.3, TUM.2
- net A0: now also C2.1, FIO_SHIELD.21, U$1.P$1; no longer C_TUM.1, FIO_SHIELD.22, TUM.1
- net A1: now also C5.1, FIO_SHIELD.22, U$1.P$4; no longer C_TA.1, FIO_SHIELD.21, TA.1
- net AREF: now also JP1.5, POT_AREF.2; no longer AREF.2, FTDI.5
- net DTR: now also JP1.1; no longer FTDI.1
- net GND: now also C2.2, C5.2, JP1.6, JUMPER_CALIB/EXEC.1, LED.K, ON/OFF.P$4, ON/OFF.P$5, POT_AREF.1, POT_THRESHOLD.1, STANDBY.GND1, STANDBY.GND2, STANDBY.P3A; no longer AREF.1, C_TA.2, C_TUM.2, FTDI.6, LED2(AMARELO).2, MODO.1, SWITCH_STANDBY.2, THRESHOLD.1
- net N$1: now also POT_THRESHOLD.2; no longer THRESHOLD.2
- net N$2: now also JUMPER_CALIB/EXEC.2; no longer SWITCH_STANDBY.1
- net N$3: now also STANDBY.P2A; no longer MODO.2
- net N$4: now also STANDBY.P1A; no longer MODO.3
- net N$7: now also LED.A; no longer LED2(AMARELO).1
- net RXI: now also JP1.3; no longer FTDI.3
- net TXO: now also JP1.2; no longer FTDI.2
Routing:
- net 3V3: track 251.5 -> 0.00 mm, vias 3 -> 0
- net GND: track 166.1 -> 0.00 mm
- net A1: track 85.6 -> 0.00 mm
- net A0: track 28.6 -> 0.00 mm
- net AREF: track 17.8 -> 0.00 mm
- net N$3: track 13.2 -> 0.00 mm
- net TXO: track 12.8 -> 0.00 mm
- net RXI: track 12.8 -> 0.00 mm
- net DTR: track 12.8 -> 0.00 mm
- net N$2: track 7.90 -> 0.00 mm, vias 2 -> 0
- net N$1: track 7.58 -> 0.00 mm
- net N$4: track 3.78 -> 0.00 mm, vias 1 -> 0
- net D10: track 3.28 -> 0.00 mm, vias 1 -> 0
- net N$7: track 3.09 -> 0.00 mm, vias 1 -> 0
- removed copper zone on layer 16, net GND
Other:
- board size 49 x 51 mm -> 55.5 x 49.5 mm
- board text removed: "BLK"
- board text removed: "GRN"

Commit message: v1_0_1
Parts:
- moved U$1 14.9 mm to (7.62, 49.5), turned to 270 degrees
- moved POT_THRESHOLD 6.48 mm to (7.62, 12.7)
- moved R5 1.80 mm to (16.5, 38.1), flipped to the bottom
- moved C5 1.80 mm to (22.9, 38.1)
- moved R4 1.80 mm to (16.5, 16.5), flipped to the bottom
- moved STANDBY 1.80 mm to (31.8, 49.5)
- moved JUMPER_CALIB/EXEC 1.80 mm to (14.0, 20.3)
- moved C2 1.80 mm to (22.9, 5.08)
- moved POT_AREF 1.80 mm to (29.2, 3.81)
- moved TUM_CALIB 1.80 mm to (17.8, 2.54)
- moved PINS_ON/OFF 1.80 mm to (11.4, 29.2)
- moved R2 1.80 mm to (38.1, 39.4), flipped to the bottom, turned to 270 degrees
- moved TA_CALIB 1.80 mm to (17.8, 25.4)
- moved JP1 1.80 mm to (41.9, 2.54)
- moved ON/OFF 1.80 mm to (1.27, 34.3)
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Routing:
- net GND: track 0.00 -> 275.7 mm, vias 0 -> 6
- net 3V3: track 0.00 -> 192.6 mm, vias 0 -> 3
- net A0: track 0.00 -> 79.6 mm, vias 0 -> 2
- net A1: track 0.00 -> 61.3 mm, vias 0 -> 2
- net N$2: track 0.00 -> 43.7 mm, vias 0 -> 2
- net N$4: track 0.00 -> 20.5 mm, vias 0 -> 2
- net N$3: track 0.00 -> 13.3 mm
- net TXO: track 0.00 -> 8.86 mm
- net DTR: track 0.00 -> 8.54 mm
- net RXI: track 0.00 -> 8.49 mm
- net AREF: track 0.00 -> 8.34 mm
- net D10: track 0.00 -> 5.79 mm
- net N$7: track 0.00 -> 5.54 mm
- net N$8: track 0.00 -> 4.73 mm
- net N$6: track 0.00 -> 4.01 mm
Other:
- board size 55.5 x 49.5 mm -> 58.1 x 52.1 mm

Commit message: v1_0_2
Routing:
- net GND: track 275.7 -> 205.1 mm, vias 6 -> 1
- net 3V3: track 192.6 -> 138.2 mm, vias 3 -> 6
- net AREF: track 8.34 -> 29.4 mm, vias 0 -> 2
- net N$1: track 0.00 -> 16.4 mm, vias 0 -> 2
- net A0: track 79.6 -> 88.1 mm
- net A1: track 61.3 -> 55.0 mm
- net N$4: track 20.5 -> 26.1 mm
- net N$3: track 13.3 -> 12.7 mm
- added copper zone on layer 1, net GND
- added copper zone on layer 16, net GND

Commit message: v1_0_3
Parts:
- removed FL1: FRAME-LETTER_BATEBIT, SparkFun-Retired:BATEBIT
Routing:
- net GND: track 205.1 -> 203.1 mm
Other:
- board size 58.1 x 52.1 mm -> 63.5 x 57.3 mm
Changed lines of the file:
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@@
 <setting verticaltext="up"/>
 </settings>
-<grid distance="0.05" unitdist="inch" unit="inch" style="lines" multiple="1" display="no" altdistance="0.025" altunitdist="inch" altunit="inch"/>
+<grid distance="1" unitdist="mm" unit="mm" style="lines" multiple="1" display="no" altdistance="0.5" altunitdist="mm" altunit="mm"/>
 <layers>
-<layer number="1" name="Top" color="4" fill="1" visible="yes" active="yes"/>
+<layer number="1" name="Top" color="4" fill="1" visible="no" active="yes"/>
 <layer number="16" name="Bottom" color="1" fill="1" visible="yes" active="yes"/>
 <layer number="17" name="Pads" color="2" fill="1" visible="yes" active="yes"/>
@@
 <layer number="19" name="Unrouted" color="6" fill="1" visible="no" active="yes"/>
 <layer number="20" name="Dimension" color="15" fill="1" visible="yes" active="yes"/>
-<layer number="21" name="tPlace" color="7" fill="1" visible="yes" active="yes"/>
-<layer number="22" name="bPlace" color="7" fill="1" visible="yes" active="yes"/>
-<layer number="23" name="tOrigins" color="15" fill="1" visible="yes" active="yes"/>
-<layer number="24" name="bOrigins" color="15" fill="1" visible="yes" active="yes"/>
-<layer number="25" name="tNames" color="7" fill="1" visible="yes" active="yes"/>
+<layer number="21" name="tPlace" color="7" fill="1" visible="no" active="yes"/>
+<layer number="22" name="bPlace" color="7" fill="1" visible="no" active="yes"/>
+<layer number="23" name="tOrigins" color="15" fill="1" visible="no" active="yes"/>
+<layer number="24" name="bOrigins" color="15" fill="1" visible="no" active="yes"/>
+<layer number="25" name="tNames" color="7" fill="1" visible="no" active="yes"/>
 <layer number="26" name="bNames" color="7" fill="1" visible="no" active="yes"/>
-<layer number="27" name="tValues" color="7" fill="1" visible="yes" active="yes"/>
+<layer number="27" name="tValues" color="7" fill="1" visible="no" active="yes"/>
 <layer number="28" name="bValues" color="7" fill="1" visible="no" active="yes"/>
 <layer number="29" name="tStop" color="7" fill="3" visible="no" active="yes"/>
@@
 <layer number="39" name="tKeepout" color="4" fill="11" visible="no" active="yes"/>
 <layer number="40" name="bKeepout" color="1" fill="11" visible="no" active="yes"/>
-<layer number="41" name="tRestrict" color="4" fill="10" visible="yes" active="yes"/>
+<layer number="41" name="tRestrict" color="4" fill="10" visible="no" active="yes"/>
 <layer number="42" name="bRestrict" color="1" fill="10" visible="no" active="yes"/>
 <layer number="43" name="vRestrict" color="2" fill="10" visible="no" active="yes"/>
@@
 <board>
 <plain>
-<wire x1="0" y1="0" x2="58.09" y2="0" width="0" layer="20"/>
-<wire x1="58.09" y1="0" x2="58.09" y2="52.06" width="0" layer="20"/>
-<wire x1="58.09" y1="52.06" x2="0" y2="52.06" width="0" layer="20"/>
-<wire x1="0" y1="52.06" x2="0" y2="0" width="0" layer="20"/>
+<wire x1="0" y1="0" x2="63.5" y2="0" width="0" layer="20"/>
+<wire x1="63.5" y1="0" x2="63.5" y2="57.3" width="0" layer="20"/>
+<wire x1="63.5" y1="57.3" x2="0" y2="57.3" width="0" layer="20"/>
+<wire x1="0" y1="57.3" x2="0" y2="0" width="0" layer="20"/>
 <hole x="3.81" y="48.26" drill="1.1"/>
 <hole x="3.81" y="45.72" drill="1.1"/>
 <hole x="3.81" y="38.1" drill="1.1"/>
 <hole x="3.81" y="40.64" drill="1.1"/>
+<hole x="50.8" y="45.72" drill="3"/>
+<hole x="48.26" y="21.59" drill="3"/>
+<hole x="3.81" y="3.81" drill="3"/>
 </plain>
 <attributes>
@@
 <element name="C5" library="SparkFun-Passives" package="CPOL-RADIAL-10UF-25V" value="" x="22.86" y="38.1"/>
 <element name="FIO_SHIELD" library="SparkFun-Boards" package="ARDUINO_FIO_SHIELD" value="ARDUINO_FIO_SHIELD&quot;" x="39.37" y="21.59" rot="R270"/>
-<element name="FL1" library="SparkFun-Retired" package="BATEBIT" value="FRAME-LETTER_BATEBIT" x="-48.26" y="10.16"/>
 <element name="JP1" library="SparkFun-Connectors" package="1X06" value="" x="41.91" y="2.54"/>
 <element name="JUMPER_CALIB/EXEC" library="SparkFun-Connectors" package="1X02" value="" x="13.97" y="20.32"/>
@@
 <wire x1="49.2125" y1="33.3375" x2="49.33" y2="33.34" width="0.8128" layer="16"/>
 <wire x1="17.78" y1="19.3675" x2="17.4625" y2="19.3675" width="0.8128" layer="16"/>
-<via x="49.2125" y="30.48" extent="1-16" drill="0.8128"/>
-<via x="20.955" y="22.5425" extent="1-16" drill="0.8128"/>
+<via x="49.2125" y="30.48" extent="1-16" drill="1.2"/>
+<via x="20.955" y="22.5425" extent="1-16" drill="1.2"/>
 </signal>
 <signal name="D10">
@@
 <wire x1="7.3025" y1="21.59" x2="7.62" y2="21.59" width="0.8128" layer="16"/>
 <wire x1="7.62" y1="21.59" x2="13.97" y2="21.59" width="0.8128" layer="16"/>
-<wire x1="5.08" y1="5.08" x2="15.5575" y2="5.08" width="0.8128" layer="16"/>
-<wire x1="5.08" y1="10.16" x2="5.08" y2="5.08" width="0.8128" layer="16"/>
+<wire x1="7.62" y1="5.08" x2="15.5575" y2="5.08" width="0.8128" layer="16"/>
+<wire x1="5.08" y1="10.16" x2="7.62" y2="5.08" width="0.8128" layer="16"/>
 <wire x1="15.5575" y1="5.08" x2="15.7748" y2="4.7776" width="0.8128" layer="16"/>
 <wire x1="21.59" y1="44.1325" x2="21.59" y2="41.91" width="0.8128" layer="16"/>
@@
 <wire x1="16.8275" y1="42.2275" x2="14.605" y2="44.45" width="0.8128" layer="16"/>
 <wire x1="16.8275" y1="42.2275" x2="17.018" y2="41.91" width="0.8128" layer="16"/>
-<via x="23.1775" y="41.91" extent="1-16" drill="0.8128"/>
+<via x="23.1775" y="41.91" extent="1-16" drill="1.2"/>
 <polygon width="0.8128" layer="1">
 <vertex x="1.27" y="50.8"/>
@@
 <wire x1="51.7525" y1="10.795" x2="51.87" y2="10.84" width="0.8128" layer="16"/>
 <wire x1="51.7525" y1="4.445" x2="51.59375" y2="4.28625" width="0.8128" layer="16"/>
-<via x="34.29" y="3.4925" extent="1-16" drill="0.8128"/>
-<via x="50.8" y="5.08" extent="1-16" drill="0.8128"/>
+<via x="34.29" y="3.4925" extent="1-16" drill="1.2"/>
+<via x="50.8" y="5.08" extent="1-16" drill="1.2"/>
 </signal>
 <signal name="RXI">
@@
 <wire x1="18.415" y1="12.065" x2="20.0025" y2="13.6525" width="0.8128" layer="1"/>
 <wire x1="18.415" y1="9.525" x2="18.415" y2="12.065" width="0.8128" layer="1"/>
-<via x="39.6875" y="6.6675" extent="1-16" drill="0.8128"/>
-<via x="48.26" y="7.62" extent="1-16" drill="0.8128"/>
-<via x="54.2925" y="17.78" extent="1-16" drill="0.8128"/>
-<via x="50.4825" y="13.97" extent="1-16" drill="0.8128"/>
-<via x="18.415" y="9.525" extent="1-16" drill="0.8128"/>
+<via x="39.6875" y="6.6675" extent="1-16" drill="1.2"/>
+<via x="48.26" y="7.62" extent="1-16" drill="1.2"/>
+<via x="54.2925" y="17.78" extent="1-16" drill="1.2"/>
+<via x="50.4825" y="13.97" extent="1-16" drill="1.2"/>
+<via x="18.415" y="9.525" extent="1-16" drill="1.2"/>
 <via x="13.6525" y="33.9725" extent="1-16" drill="0.8128"/>
 </signal>
@@
 <wire x1="39.0525" y1="10.795" x2="39.17" y2="10.84" width="0.8128" layer="16"/>
 <wire x1="22.5425" y1="7.9375" x2="22.5425" y2="7.3025" width="0.8128" layer="16"/>
-<via x="6.6675" y="37.1475" extent="1-16" drill="0.8128"/>
-<via x="13.335" y="7.9375" extent="1-16" drill="0.8128"/>
+<via x="6.6675" y="37.1475" extent="1-16" drill="1.2"/>
+<via x="13.335" y="7.9375" extent="1-16" drill="1.2"/>
 </signal>
 <signal name="A1">
@@
 <wire x1="17.30375" y1="31.27375" x2="36.5125" y2="12.065" width="0.8128" layer="16"/>
 <wire x1="36.5125" y1="11.1125" x2="36.63" y2="10.84" width="0.8128" layer="16"/>
-<via x="14.605" y="40.64" extent="1-16" drill="0.8128"/>
-<via x="19.05" y="39.6875" extent="1-16" drill="0.8128"/>
+<via x="14.605" y="40.64" extent="1-16" drill="1.2"/>
+<via x="19.05" y="39.6875" extent="1-16" drill="1.2"/>
 </signal>
 <signal name="N$1">
@@
 <wire x1="21.2725" y1="11.1125" x2="21.2725" y2="13.97" width="0.8128" layer="16"/>
 <wire x1="21.2725" y1="11.1125" x2="21.39" y2="10.84" width="0.8128" layer="16"/>
-<via x="13.335" y="15.875" extent="1-16" drill="0.8128"/>
-<via x="19.3675" y="15.875" extent="1-16" drill="0.8128"/>
+<via x="13.335" y="15.875" extent="1-16" drill="1.2"/>
+<via x="19.3675" y="15.875" extent="1-16" drill="1.2"/>
 </signal>
 <signal name="N$4">
@@
 <wire x1="27.6225" y1="44.1325" x2="28.2575" y2="43.4975" width="0.8128" layer="16"/>
 <wire x1="27.6225" y1="44.1325" x2="27.432" y2="44.196" width="0.8128" layer="16"/>
-<via x="13.6525" y="38.1" extent="1-16" drill="0.8128"/>
-<via x="27.94" y="35.8775" extent="1-16" drill="0.8128"/>
+<via x="13.6525" y="38.1" extent="1-16" drill="1.2"/>
+<via x="27.94" y="35.8775" extent="1-16" drill="1.2"/>
 </signal>
 <signal name="N$3">
@@
 <wire x1="7.62" y1="27.94" x2="7.9375" y2="27.94" width="0.8128" layer="16"/>
 </signal>
+<signal name="N$5">
+<via x="3" y="55" extent="1-16" drill="0.8" shape="octagon"/>
+</signal>
+<signal name="N$9">
+<via x="61" y="55" extent="1-16" drill="0.8" shape="octagon"/>
+</signal>
+<signal name="N$10">
+<via x="61" y="3" extent="1-16" drill="0.8" shape="octagon"/>
+</signal>
 </signals>

Commit message: v1_0_4
Connections:
- removed net 3.3V: POT_THRESHOLD.3
- net 3V3: now also POT_THRESHOLD.3
Routing:
- net 3V3: track 138.2 -> 155.7 mm, vias 6 -> 7
