File: PCB/TumTa.sch (EAGLE design)
At the start: 16 parts

Commit message: v0_2_4
Parts:
- added C3, C4, C5, C6: (no value), SparkFun-Passives:CAP_POLPTH2
Connections:
- net N$4 renamed D9
- net N$5 renamed D10
- removed net 3.3V: CAL_TA.CCW, CAL_TUM.CCW
- removed net N$1: FIO_SHIELD.D8, R4.2
- removed net N$11: FIO_SHIELD.A3
- removed net N$12: C2.+, CAL_TA.WIPER, TA.ESQ
- removed net N$9: C1.+, CAL_TUM.WIPER, FIO_SHIELD.A1, TUM.ESQ
- new net A0: C1.+, C2.+, C3.+, CAL_TUM.WIPER, FIO_SHIELD.A0, TUM.ESQ
- new net A1: C4.+, C5.+, C6.+, CAL_TA.WIPER, FIO_SHIELD.A1, TA.ESQ
- new net D6: FIO_SHIELD.D6*, R4.2
- net 3V3: now also CAL_TA.CCW, CAL_TUM.CCW, FIO_SHIELD.3V3@1
- net GND: now also C3.-, C4.-, C5.-, C6.-, FIO_SHIELD.GND@2
Other:
- note added: "0.2.4"
- note added: "Versao sem auto-route"
- note removed: "0.2.2"
- moved on the sheet: C1, C2, CAL_TA, CAL_TUM, LED1(VERDE), LED2(AMARELO), R1, R2, R4, SWITCH_STANDBY, TA, TUM

Commit message: v0_2_10
Parts:
- removed C1, C3, C4, C6: (no value), SparkFun-Passives:CAP_POLPTH2
- removed CAL_TA, CAL_TETO, CAL_TUM: TRIMPOT_MULTIVOLTAS, SparkFun-Electromechanical:TRIMPOT_MULTIVOLTAS
- removed LED1(VERDE): SCREWTERMINAL-25MM, SparkFun-Connectors:SCREWTERMINAL-25MM
- removed R1: 100, SparkFun-Resistors:10OHM-1/10W-1%(0603)SMD
- added AREF, R3: (no value), SparkFun-Electromechanical:TRIMPOTBR
- added R5: 4.7K, SparkFun-Resistors:4.7KOHM-1/10W-1%(0603)
- added S1: (no value), SparkFun-Electromechanical:SWITCH-SPDTPTH
- added TA_CALIB, TUM_CALIB: TRIMPOT_MULTIVOLTAS, SparkFun-Electromechanical:TRIMPOT_MULTIVOLTAS
Connections:
- removed net D6: FIO_SHIELD.D6*, R4.2
- removed net D9: FIO_SHIELD.D9*, R1.2
- new net N$1: FIO_SHIELD.A7, R3.WIPER
- new net N$4: R5.2, S1.S
- net 3V3: now also AREF.CW, R3.CW, R4.2, R5.1, TA.DIR, TA_CALIB.CW, TUM.DIR, TUM_CALIB.CW; no longer CAL_TA.CCW, CAL_TETO.CW, CAL_TUM.CCW
- net A0: now also TUM_CALIB.WIPER; no longer C1.+, C3.+, CAL_TUM.WIPER
- net A1: now also TA_CALIB.WIPER; no longer C4.+, C6.+, CAL_TA.WIPER
- net AREF: now also AREF.WIPER; no longer CAL_TETO.WIPER
- net D10: now also FIO_SHIELD.D6*; no longer FIO_SHIELD.D10*
- net GND: now also AREF.CCW, R3.CCW, S1.O, TA_CALIB.CCW, TUM_CALIB.CCW; no longer C1.-, C3.-, C4.-, C6.-, CAL_TETO.CCW, LED1(VERDE).DIR, TA.DIR, TUM.DIR
- net N$2: now also FIO_SHIELD.D2
- net N$3: now also FIO_SHIELD.D12, S1.P; no longer LED1(VERDE).ESQ, R1.1
Other:
- note added: "0.2.9 unrouted"
- note removed: "0.2.4"
- note removed: "Versao sem auto-route"
- moved on the sheet: C2, C5, JP1, LED2(AMARELO), R2, R4, SWITCH_STANDBY

Commit message: v0_2_3
Parts:
- removed AREF, R3: (no value), SparkFun-Electromechanical:TRIMPOTBR
- removed C5: (no value), SparkFun-Passives:CAP_POLPTH2
- removed R5: 4.7K, SparkFun-Resistors:4.7KOHM-1/10W-1%(0603)
- removed S1: (no value), SparkFun-Electromechanical:SWITCH-SPDTPTH
- removed TA_CALIB, TUM_CALIB: TRIMPOT_MULTIVOLTAS, SparkFun-Electromechanical:TRIMPOT_MULTIVOLTAS
- added C1: (no value), SparkFun-Passives:CAP_POLPTH2
- added CAL_TA, CAL_TETO, CAL_TUM: TRIMPOT_MULTIVOLTAS, SparkFun-Electromechanical:TRIMPOT_MULTIVOLTAS
- added LED1(VERDE): SCREWTERMINAL-25MM, SparkFun-Connectors:SCREWTERMINAL-25MM
- added R1: 100, SparkFun-Resistors:10OHM-1/10W-1%(0603)SMD
Connections:
- removed net A0: C2.+, FIO_SHIELD.A0, TUM.ESQ, TUM_CALIB.WIPER
- removed net A1: C5.+, FIO_SHIELD.A1, TA.ESQ, TA_CALIB.WIPER
- removed net D10: FIO_SHIELD.D6*, R2.2
- new net 3.3V: CAL_TA.CCW, CAL_TUM.CCW
- new net N$11: FIO_SHIELD.A3
- new net N$12: C2.+, CAL_TA.WIPER, TA.ESQ
- new net N$5: FIO_SHIELD.D10*, R2.2
- new net N$9: C1.+, CAL_TUM.WIPER, FIO_SHIELD.A1, TUM.ESQ
- net 3V3: now also CAL_TETO.CW; no longer AREF.CW, FIO_SHIELD.3V3@1, R3.CW, R4.2, R5.1, TA.DIR, TA_CALIB.CW, TUM.DIR, TUM_CALIB.CW
- net AREF: now also CAL_TETO.WIPER; no longer AREF.WIPER
- net GND: now also C1.-, CAL_TETO.CCW, LED1(VERDE).DIR, TA.DIR, TUM.DIR; no longer AREF.CCW, C5.-, FIO_SHIELD.GND@2, R3.CCW, S1.O, TA_CALIB.CCW, TUM_CALIB.CCW
- net N$1: now also FIO_SHIELD.D6*, R4.2; no longer FIO_SHIELD.A7, R3.WIPER
- net N$2: no longer FIO_SHIELD.D2
- net N$3: now also LED1(VERDE).ESQ, R1.1; no longer FIO_SHIELD.D12, S1.P
- net N$4: now also FIO_SHIELD.D9*, R1.2; no longer R5.2, S1.S
Other:
- note added: "0.2.2"
- note removed: "0.2.9 unrouted"
- moved on the sheet: C2, JP1, LED2(AMARELO), R2, R4, SWITCH_STANDBY, TA, TUM

Commit message: v0_2_4
Parts:
- added C3, C4, C5, C6: (no value), SparkFun-Passives:CAP_POLPTH2
Connections:
- net N$1 renamed D6
- net N$4 renamed D9
- net N$5 renamed D10
- removed net 3.3V: CAL_TA.CCW, CAL_TUM.CCW
- removed net N$11: FIO_SHIELD.A3
- removed net N$12: C2.+, CAL_TA.WIPER, TA.ESQ
- removed net N$9: C1.+, CAL_TUM.WIPER, FIO_SHIELD.A1, TUM.ESQ
- new net A0: C1.+, C2.+, C3.+, CAL_TUM.WIPER, FIO_SHIELD.A0, TUM.ESQ
- new net A1: C4.+, C5.+, C6.+, CAL_TA.WIPER, FIO_SHIELD.A1, TA.ESQ
- net 3V3: now also CAL_TA.CCW, CAL_TUM.CCW, FIO_SHIELD.3V3@1
- net GND: now also C3.-, C4.-, C5.-, C6.-, FIO_SHIELD.GND@2
Other:
- note added: "0.2.4"
- note added: "Versao sem auto-route"
- note removed: "0.2.2"
- moved on the sheet: C1, C2, CAL_TA, CAL_TUM, LED1(VERDE), LED2(AMARELO), R1, R2, TA, TUM

Commit message: v0_2_5
Other:
- note added: "0.2.5"
- note added: "Versao com trilhas"
- note removed: "0.2.4"
- note removed: "Versao sem auto-route"
Changed lines of the file:
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@@
 <plain>
 <text x="48.26" y="-83.82" size="2.54" layer="94" font="fixed">JOÃO TRAGTENBERG</text>
-<text x="120.65" y="-84.328" size="2.54" layer="94" font="fixed">0.2.4</text>
-<text x="81.28" y="-73.66" size="1.778" layer="94" font="vector">Versao sem auto-route</text>
+<text x="120.65" y="-84.328" size="2.54" layer="94" font="fixed">0.2.5</text>
+<text x="81.28" y="-73.66" size="1.778" layer="94" font="vector">Versao com trilhas</text>
 </plain>
 <instances>

Commit message: v0_2_6
Other:
- note added: "0.2.6"
- note added: "Versao com rats nests"
- note removed: "0.2.5"
- note removed: "Versao com trilhas"
Changed lines of the file:
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@@
 <plain>
 <text x="48.26" y="-83.82" size="2.54" layer="94" font="fixed">JOÃO TRAGTENBERG</text>
-<text x="120.65" y="-84.328" size="2.54" layer="94" font="fixed">0.2.5</text>
-<text x="81.28" y="-73.66" size="1.778" layer="94" font="vector">Versao com trilhas</text>
+<text x="120.65" y="-84.328" size="2.54" layer="94" font="fixed">0.2.6</text>
+<text x="81.28" y="-73.66" size="1.778" layer="94" font="vector">Versao com rats nests</text>
 </plain>
 <instances>

Commit message: v0_2_7
Parts:
- removed CAL_TETO: TRIMPOT_MULTIVOLTAS, SparkFun-Electromechanical:TRIMPOT_MULTIVOLTAS
- added R3: (no value), SparkFun-Electromechanical:TRIMPOTPTH
Connections:
- net 3V3: now also R3.CW, TA.DIR, TUM.DIR; no longer CAL_TA.CCW, CAL_TETO.CW, CAL_TUM.CCW
- net AREF: now also R3.WIPER; no longer CAL_TETO.WIPER
- net GND: now also CAL_TA.CCW, CAL_TUM.CCW, R3.CCW; no longer CAL_TETO.CCW, TA.DIR, TUM.DIR
Other:
- note added: "0.2.7 unrouted"
- note added: "Versao com trilhas"
- note removed: "0.2.6"
- note removed: "Versao com rats nests"
- moved on the sheet: JP1
Changed lines of the file:
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@@
 </variantdefs>
 <classes>
-<class number="0" name="default" width="0" drill="0">
+<class number="0" name="default" width="0.6096" drill="0">
 </class>
 </classes>
@@
 <part name="GND3" library="SparkFun-Aesthetics" deviceset="GND" device=""/>
 <part name="GND4" library="SparkFun-Aesthetics" deviceset="GND" device=""/>
-<part name="CAL_TETO" library="SparkFun-Electromechanical" deviceset="TRIMPOT_MULTIVOLTAS" device=""/>
 <part name="JP1" library="SparkFun-Connectors" deviceset="ARDUINO_SERIAL_PROGRAM" device="PTH"/>
 <part name="GND5" library="SparkFun-Aesthetics" deviceset="GND" device=""/>
 <part name="SUPPLY1" library="SparkFun-Aesthetics" deviceset="3.3V" device=""/>
 <part name="TUM" library="SparkFun-Connectors" deviceset="SCREWTERMINAL-2" device="5MM"/>
-<part name="SUPPLY2" library="SparkFun-Aesthetics" deviceset="3.3V" device=""/>
-<part name="GND8" library="SparkFun-Aesthetics" deviceset="GND" device=""/>
 <part name="CAL_TUM" library="SparkFun-Electromechanical" deviceset="TRIMPOT_MULTIVOLTAS" device=""/>
 <part name="TA" library="SparkFun-Connectors" deviceset="SCREWTERMINAL-2" device="5MM"/>
-<part name="SUPPLY3" library="SparkFun-Aesthetics" deviceset="3.3V" device=""/>
-<part name="GND9" library="SparkFun-Aesthetics" deviceset="GND" device=""/>
 <part name="CAL_TA" library="SparkFun-Electromechanical" deviceset="TRIMPOT_MULTIVOLTAS" device=""/>
 <part name="C1" library="SparkFun-Passives" deviceset="CAP_POL" device="PTH2"/>
@@
 <part name="GND1" library="SparkFun-Aesthetics" deviceset="GND" device=""/>
 <part name="GND11" library="SparkFun-Aesthetics" deviceset="GND" device=""/>
+<part name="GND6" library="SparkFun-Aesthetics" deviceset="GND" device=""/>
+<part name="SUPPLY4" library="SparkFun-Aesthetics" deviceset="3.3V" device=""/>
+<part name="SUPPLY5" library="SparkFun-Aesthetics" deviceset="3.3V" device=""/>
+<part name="GND7" library="SparkFun-Aesthetics" deviceset="GND" device=""/>
+<part name="R3" library="SparkFun-Electromechanical" deviceset="TRIMPOT" device="PTH"/>
 </parts>
 <sheets>
@@
 <plain>
 <text x="48.26" y="-83.82" size="2.54" layer="94" font="fixed">JOÃO TRAGTENBERG</text>
-<text x="120.65" y="-84.328" size="2.54" layer="94" font="fixed">0.2.6</text>
-<text x="81.28" y="-73.66" size="1.778" layer="94" font="vector">Versao com rats nests</text>
+<text x="120.65" y="-84.328" size="2.54" layer="94" font="fixed">0.2.7 unrouted</text>
+<text x="81.28" y="-73.66" size="1.778" layer="94" font="vector">Versao com trilhas</text>
 </plain>
 <instances>
@@
 <instance part="GND3" gate="1" x="-43.18" y="-15.24"/>
 <instance part="GND4" gate="1" x="-43.18" y="-2.54"/>
-<instance part="CAL_TETO" gate="G$1" x="50.8" y="10.16"/>
-<instance part="JP1" gate="G$1" x="83.82" y="15.24" rot="MR0"/>
+<instance part="JP1" gate="G$1" x="104.14" y="35.56" rot="MR0"/>
 <instance part="GND5" gate="1" x="43.18" y="7.62"/>
 <instance part="SUPPLY1" gate="G$1" x="68.58" y="10.16"/>
 <instance part="TUM" gate="G$1" x="93.98" y="2.54" rot="MR0"/>
-<instance part="SUPPLY2" gate="G$1" x="33.02" y="-5.08"/>
-<instance part="GND8" gate="1" x="86.36" y="-2.54"/>
 <instance part="CAL_TUM" gate="G$1" x="40.64" y="-5.08"/>
 <instance part="TA" gate="G$1" x="93.98" y="-17.78" rot="MR0"/>
-<instance part="SUPPLY3" gate="G$1" x="33.02" y="-25.4"/>
-<instance part="GND9" gate="1" x="86.36" y="-22.86"/>
 <instance part="CAL_TA" gate="G$1" x="40.64" y="-25.4"/>
 <instance part="C1" gate="G$1" x="60.96" y="-2.54"/>
@@
 <instance part="GND1" gate="1" x="68.58" y="-35.56"/>
 <instance part="GND11" gate="1" x="68.58" y="-12.7"/>
+<instance part="GND6" gate="1" x="33.02" y="-7.62"/>
+<instance part="SUPPLY4" gate="G$1" x="83.82" y="-5.08"/>
+<instance part="SUPPLY5" gate="G$1" x="83.82" y="-27.94"/>
+<instance part="GND7" gate="1" x="33.02" y="-27.94"/>
+<instance part="R3" gate="R?" x="50.8" y="10.16"/>
 </instances>
 <busses>
@@
 <segment>
 <pinref part="JP1" gate="G$1" pin="GND"/>
-<wire x1="78.74" y1="22.86" x2="76.2" y2="22.86" width="0.1524" layer="91"/>
-<label x="76.2" y="22.86" size="1.778" layer="95"/>
+<wire x1="99.06" y1="43.18" x2="96.52" y2="43.18" width="0.1524" layer="91"/>
+<label x="96.52" y="43.18" size="1.778" layer="95"/>
 </segment>
 <segment>
@@
 </segment>
 <segment>
-<pinref part="CAL_TETO" gate="G$1" pin="CCW"/>
 <pinref part="GND5" gate="1" pin="GND"/>
 <wire x1="45.72" y1="10.16" x2="43.18" y2="10.16" width="0.1524" layer="91"/>
-</segment>
-<segment>
-<pinref part="TUM" gate="G$1" pin="DIR"/>
-<wire x1="88.9" y1="0" x2="86.36" y2="0" width="0.1524" layer="91"/>
-<pinref part="GND8" gate="1" pin="GND"/>
-</segment>
-<segment>
-<wire x1="88.9" y1="-20.32" x2="86.36" y2="-20.32" width="0.1524" layer="91"/>
-<pinref part="TA" gate="G$1" pin="DIR"/>
-<pinref part="GND9" gate="1" pin="GND"/>
+<pinref part="R3" gate="R?" pin="CCW"/>
 </segment>
 <segment>
@@
 <pinref part="C1" gate="G$1" pin="-"/>
 </segment>
+<segment>
+<pinref part="CAL_TA" gate="G$1" pin="CCW"/>
+<pinref part="GND7" gate="1" pin="GND"/>
+<wire x1="35.56" y1="-25.4" x2="33.02" y2="-25.4" width="0.1524" layer="91"/>
+</segment>
+<segment>
+<pinref part="CAL_TUM" gate="G$1" pin="CCW"/>
+<pinref part="GND6" gate="1" pin="GND"/>
+<wire x1="35.56" y1="-5.08" x2="33.02" y2="-5.08" width="0.1524" layer="91"/>
+</segment>
 </net>
 <net name="AREF" class="0">
 <segment>
 <pinref part="JP1" gate="G$1" pin="CTS"/>
-<wire x1="78.74" y1="20.32" x2="76.2" y2="20.32" width="0.1524" layer="91"/>
-<label x="76.2" y="20.32" size="1.778" layer="95"/>
+<wire x1="99.06" y1="40.64" x2="96.52" y2="40.64" width="0.1524" layer="91"/>
+<label x="96.52" y="40.64" size="1.778" layer="95"/>
 </segment>
 <segment>
 <pinref part="FIO_SHIELD" gate="G$1" pin="AREF"/>
 <label x="20.32" y="15.24" size="1.778" layer="95"/>
-<pinref part="CAL_TETO" gate="G$1" pin="WIPER"/>
 <wire x1="17.78" y1="15.24" x2="50.8" y2="15.24" width="0.1524" layer="91"/>
+<pinref part="R3" gate="R?" pin="WIPER"/>
 </segment>
 </net>
@@
 <segment>
 <pinref part="JP1" gate="G$1" pin="TXO"/>
-<wire x1="78.74" y1="15.24" x2="76.2" y2="15.24" width="0.1524" layer="91"/>
-<label x="76.2" y="15.24" size="1.778" layer="95"/>
+<wire x1="99.06" y1="35.56" x2="96.52" y2="35.56" width="0.1524" layer="91"/>
+<label x="96.52" y="35.56" size="1.778" layer="95"/>
 </segment>
 <segment>
@@
 <segment>
 <pinref part="JP1" gate="G$1" pin="RXI"/>
-<wire x1="78.74" y1="12.7" x2="76.2" y2="12.7" width="0.1524" layer="91"/>
-<label x="76.2" y="12.7" size="1.778" layer="95"/>
+<wire x1="99.06" y1="33.02" x2="96.52" y2="33.02" width="0.1524" layer="91"/>
+<label x="96.52" y="33.02" size="1.778" layer="95"/>
 </segment>
 <segment>
@@
 <segment>
 <pinref part="JP1" gate="G$1" pin="DTR"/>
-<wire x1="78.74" y1="10.16" x2="76.2" y2="10.16" width="0.1524" layer="91"/>
-<label x="76.2" y="10.16" size="1.778" layer="95"/>
+<wire x1="99.06" y1="30.48" x2="96.52" y2="30.48" width="0.1524" layer="91"/>
+<label x="96.52" y="30.48" size="1.778" layer="95"/>
 </segment>
 <segment>
@@
 <segment>
 <pinref part="JP1" gate="G$1" pin="VCC"/>
-<wire x1="78.74" y1="17.78" x2="76.2" y2="17.78" width="0.1524" layer="91"/>
-<label x="76.2" y="17.78" size="1.778" layer="95"/>
-</segment>
-<segment>
-<pinref part="CAL_TETO" gate="G$1" pin="CW"/>
+<wire x1="99.06" y1="38.1" x2="96.52" y2="38.1" width="0.1524" layer="91"/>
+<label x="96.52" y="38.1" size="1.778" layer="95"/>
+</segment>
+<segment>
 <pinref part="SUPPLY1" gate="G$1" pin="3.3V"/>
 <wire x1="55.88" y1="10.16" x2="68.58" y2="10.16" width="0.1524" layer="91"/>
-</segment>
-<segment>
-<wire x1="35.56" y1="-5.08" x2="33.02" y2="-5.08" width="0.1524" layer="91"/>
-<pinref part="SUPPLY2" gate="G$1" pin="3.3V"/>
-<pinref part="CAL_TUM" gate="G$1" pin="CCW"/>
-</segment>
-<segment>
-<pinref part="SUPPLY3" gate="G$1" pin="3.3V"/>
-<pinref part="CAL_TA" gate="G$1" pin="CCW"/>
-<wire x1="33.02" y1="-25.4" x2="35.56" y2="-25.4" width="0.1524" layer="91"/>
+<pinref part="R3" gate="R?" pin="CW"/>
 </segment>
 <segment>
@@
 <label x="-22.86" y="17.78" size="1.778" layer="95" font="vector"/>
 </segment>
-</net>
+<segment>
+<pinref part="TUM" gate="G$1" pin="DIR"/>
+<wire x1="88.9" y1="0" x2="88.9" y2="-5.08" width="0.1524" layer="91"/>
+<pinref part="SUPPLY4" gate="G$1" pin="3.3V"/>
+<wire x1="88.9" y1="-5.08" x2="83.82" y2="-5.08" width="0.1524" layer="91"/>
+</segment>
+<segment>
+<pinref part="TA" gate="G$1" pin="DIR"/>
+<wire x1="88.9" y1="-20.32" x2="88.9" y2="-27.94" width="0.1524" layer="91"/>
+<pinref part="SUPPLY5" gate="G$1" pin="3.3V"/>
+<wire x1="88.9" y1="-27.94" x2="83.82" y2="-27.94" width="0.1524" layer="91"/>
+</segment>
+</net>

Commit message: v0_2_8
Parts:
- removed CAL_TA, CAL_TUM: TRIMPOT_MULTIVOLTAS, SparkFun-Electromechanical:TRIMPOT_MULTIVOLTAS
- removed R3: (no value), SparkFun-Electromechanical:TRIMPOTPTH
- added AREF, TA_CALIB, TUM_CALIB: (no value), SparkFun-Electromechanical:TRIMPOTBR
Connections:
- new net 3.3V: TA.DIR, TA_CALIB.CW, TUM.DIR, TUM_CALIB.CW
- net 3V3: now also AREF.CW; no longer R3.CW, TA.DIR, TUM.DIR
- net A0: now also TUM_CALIB.WIPER; no longer CAL_TUM.WIPER
- net A1: now also TA_CALIB.WIPER; no longer CAL_TA.WIPER
- net AREF: now also AREF.WIPER; no longer R3.WIPER
- net GND: now also AREF.CCW, TA_CALIB.CCW, TUM_CALIB.CCW; no longer CAL_TA.CCW, CAL_TUM.CCW, R3.CCW
Other:
- note added: "0.2.8"
- note removed: "0.2.7 unrouted"
- moved on the sheet: C1, C2, C3, C4, C5, C6
