File: PCB/TumTa.sch (EAGLE design)
At the start: 20 parts

Commit message: v0_2_9
Parts:
- removed C1, C2, C3, C4, C5, C6: (no value), SparkFun-Passives:CAP_POLPTH2
- removed FL1: FRAME-LETTER_BATEBIT, SparkFun-Retired:FRAME-LETTER_BATEBIT
- removed LED1(VERDE): SCREWTERMINAL-25MM, SparkFun-Connectors:SCREWTERMINAL-25MM
- removed R1: 100, SparkFun-Resistors:10OHM-1/10W-1%(0603)SMD
- added C_TA, C_TUM: (no value), SparkFun-Passives:CAP_POLPTH2
- added MODO: (no value), SparkFun-Electromechanical:SWITCH-SPDTPTH
- added R5: 4.7K, SparkFun-Resistors:4.7KOHM-1/10W-1%(0603)
- added THRESHOLD: (no value), SparkFun-Electromechanical:TRIMPOTBR
- TA_CALIB, TUM_CALIB: value (none) -> TRIMPOT_MULTIVOLTAS; device SparkFun-Electromechanical:TRIMPOTBR -> SparkFun-Electromechanical:TRIMPOT_MULTIVOLTAS
- renumbered JP1 to FTDI
Connections:
- removed net 3.3V: TA.DIR, TA_CALIB.CW, TUM.DIR, TUM_CALIB.CW
- removed net D6: FIO_SHIELD.D6*, R4.2
- removed net D9: FIO_SHIELD.D9*, R1.2
- new net N$1: FIO_SHIELD.A7, THRESHOLD.WIPER
- new net N$4: MODO.S, R5.2
- net 3V3: now also R4.2, R5.1, TA.DIR, TA_CALIB.CW, THRESHOLD.CW, TUM.DIR, TUM_CALIB.CW
- net A0: now also C_TUM.+, FIO_SHIELD.A1; no longer C1.+, C2.+, C3.+, FIO_SHIELD.A0
- net A1: now also C_TA.+, FIO_SHIELD.A0; no longer C4.+, C5.+, C6.+, FIO_SHIELD.A1
- net D10: now also FIO_SHIELD.D6*; no longer FIO_SHIELD.D10*
- net GND: now also C_TA.-, C_TUM.-, MODO.O, THRESHOLD.CCW; no longer C1.-, C2.-, C3.-, C4.-, C5.-, C6.-, LED1(VERDE).DIR
- net N$2: now also FIO_SHIELD.D2
- net N$3: now also FIO_SHIELD.D12, MODO.P; no longer LED1(VERDE).ESQ, R1.1
Other:
- note added: "0.2.9 unrouted"
- note removed: "0.2.8"
- note removed: "Versao com trilhas"
- moved on the sheet: LED2(AMARELO), R2, R4, SWITCH_STANDBY, TA, TUM

Commit message: v1_0_0
Parts:
- removed AREF: (no value), SparkFun-Electromechanical:TRIMPOTBR
- removed C_TA, C_TUM: (no value), SparkFun-Passives:CAP_POLPTH2
- removed LED2(AMARELO), SWITCH_STANDBY, TA, TUM: SCREWTERMINAL-25MM, SparkFun-Connectors:SCREWTERMINAL-25MM
- removed MODO: (no value), SparkFun-Electromechanical:SWITCH-SPDTPTH
- added C2, C5: (no value), SparkFun-Passives:CAP_POLPTH2
- added FL1: FRAME-LETTER_BATEBIT, SparkFun-Retired:FRAME-LETTER_BATEBIT
- added JUMPER_CALIB/EXEC, PINS_ON/OFF: (no value), SparkFun-Connectors:M02PTH
- added LED: (no value), SparkFun-LED:LED-GREEN5MM_THRU
- added ON/OFF: SWITCH, SparkFun-Electromechanical:SWITCH-SPDT-COM-GND3PIN
- added POT_AREF: TRIMPOT_MULTIVOLTAS, SparkFun-Electromechanical:TRIMPOT_MULTIVOLTAS
- added STANDBY: SWITCH, SparkFun-Electromechanical:SWITCH-SPDT-COM-GND6PIN
- added U$1: SCREWTERMINAL-5, SparkFun-Connectors:SCREWTERMINAL-5
- renumbered FTDI to JP1, THRESHOLD to POT_THRESHOLD
Connections:
- new net 3.3V: POT_THRESHOLD.CW
- new net N$6: ON/OFF.O, PINS_ON/OFF.2
- new net N$8: ON/OFF.P, PINS_ON/OFF.1
- net 3V3: now also POT_AREF.CW, U$1.2, U$1.5; no longer AREF.CW, POT_THRESHOLD.CW, TA.DIR, TUM.DIR
- net A0: now also C2.+, FIO_SHIELD.A0, U$1.1; no longer C_TUM.+, FIO_SHIELD.A1, TUM.ESQ
- net A1: now also C5.+, FIO_SHIELD.A1, U$1.4; no longer C_TA.+, FIO_SHIELD.A0, TA.ESQ
- net AREF: now also POT_AREF.WIPER; no longer AREF.WIPER
- net GND: now also C2.-, C5.-, JUMPER_CALIB/EXEC.1, LED.C, ON/OFF.GND, ON/OFF.GND1, POT_AREF.CCW, STANDBY.GND, STANDBY.GND1, STANDBY.S; no longer AREF.CCW, C_TA.-, C_TUM.-, LED2(AMARELO).DIR, MODO.O, SWITCH_STANDBY.DIR
- net N$2: now also JUMPER_CALIB/EXEC.2; no longer SWITCH_STANDBY.ESQ
- net N$3: now also STANDBY.P; no longer MODO.P
- net N$4: now also STANDBY.O; no longer MODO.S
- net N$7: now also LED.A; no longer LED2(AMARELO).ESQ
Other:
- note added: "1.0.0"
- note added: "ta"
- note added: "tum"
- note removed: "0.2.9 unrouted"
- moved on the sheet: R5, TA_CALIB, TUM_CALIB

Commit message: v1_0_3
Parts:
- removed FL1: FRAME-LETTER_BATEBIT, SparkFun-Retired:FRAME-LETTER_BATEBIT
Changed lines of the file:
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@@
 <part name="GND5" library="SparkFun-Aesthetics" deviceset="GND" device=""/>
 <part name="SUPPLY1" library="SparkFun-Aesthetics" deviceset="3.3V" device=""/>
-<part name="FL1" library="SparkFun-Retired" deviceset="FRAME-LETTER_BATEBIT" device=""/>
 <part name="C2" library="SparkFun-Passives" deviceset="CAP_POL" device="PTH2"/>
 <part name="C5" library="SparkFun-Passives" deviceset="CAP_POL" device="PTH2"/>
@@
 <instance part="GND5" gate="1" x="38.1" y="7.62"/>
 <instance part="SUPPLY1" gate="G$1" x="68.58" y="10.16"/>
-<instance part="FL1" gate="G$1" x="-116.84" y="-91.44"/>
-<instance part="FL1" gate="G$2" x="30.734" y="-91.44"/>
 <instance part="C2" gate="G$1" x="48.26" y="-2.54"/>
 <instance part="C5" gate="G$1" x="48.26" y="-25.4"/>

Commit message: v1_0_4
Connections:
- removed net 3.3V: POT_THRESHOLD.CW
- net 3V3: now also POT_THRESHOLD.CW
Changed lines of the file:
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@@
 <wire x1="-60.96" y1="-22.86" x2="-68.58" y2="-22.86" width="0.1524" layer="91"/>
+</segment>
+<segment>
+<pinref part="POT_THRESHOLD" gate="R?" pin="CW"/>
+<pinref part="SUPPLY3" gate="G$1" pin="3.3V"/>
+<wire x1="38.1" y1="-43.18" x2="48.26" y2="-43.18" width="0.1524" layer="91"/>
 </segment>
 </net>
@@
 </segment>
 </net>
-<net name="3.3V" class="0">
-<segment>
-<pinref part="POT_THRESHOLD" gate="R?" pin="CW"/>
-<pinref part="SUPPLY3" gate="G$1" pin="3.3V"/>
-<wire x1="38.1" y1="-43.18" x2="48.26" y2="-43.18" width="0.1524" layer="91"/>
-</segment>
-</net>
